Commit message: Changes: - Updated origin of `base_joint` to move the entire pendulum above ground. - Added `inertial_macros.xacro` for inertial calculations. - Renamed `robot.urdf` -> `robot.urdf.xacro` for xacro compatibility.

File: pendulum_description/description/robot.urdf.xacro (robot description, xacro)
@@ -1,8 +1,10 @@
 <?xml version="1.0"?>
 <robot xmlns:xacro="http://www.ros.org/wiki/xacro" name="pendulum">
+  <xacro:include filename="inertial_macros.xacro" />
   <link name="base_link" />
   <joint name="base_joint" type="continuous">
     <parent link="base_link" />
     <child link="pendulum_arm" />
+    <origin xyz="0 0 0.35" />
   </joint>
   <link name="pendulum_arm">
@@ -22,5 +24,7 @@
       </geometry>
     </collision>
-    <!-- Inertial properties can be added here -->
+    <xacro:inertial_cylinder mass="0.5" radius="0.02" length="0.2">
+      <origin xyz="0.0 0.0 -0.1" />
+    </xacro:inertial_cylinder>
   </link>
   <joint name="arm_to_bob" type="fixed">
@@ -43,5 +47,7 @@
       </geometry>
     </collision>
-    <!-- Inertial properties can be added here -->
+    <xacro:inertial_sphere mass="1.0" radius="0.05">
+      <origin xyz="0 0 0" />
+    </xacro:inertial_sphere>
   </link>
 </robot>

Commit message: Added sim support: - The new pkg `pendulum_sim` now has `launch/gazebo.launch.py` for simulation of the pendulum. - Added `ros_gz_bridge.yaml` for relaying gz topics to ros. - Minor modifications to `robot.urdf.xacro` to add values to `base_link` (needed for gz) - Copied over `setup.py` for easier file compilations.

File: pendulum_description/description/robot.urdf.xacro (robot description, xacro)
@@ -2,5 +2,24 @@
 <robot xmlns:xacro="http://www.ros.org/wiki/xacro" name="pendulum">
   <xacro:include filename="inertial_macros.xacro" />
-  <link name="base_link" />
+  <link name="base_link">
+    <visual>
+      <origin xyz="0.0 0.0 0.025" />
+      <geometry>
+        <box size="0.1 0.1 0.05" />
+      </geometry>
+      <material name="gray">
+        <color rgba="0.5 0.5 0.5 1" />
+      </material>
+    </visual>
+    <collision>
+      <origin xyz="0.0 0.0 0.025" />
+      <geometry>
+        <box size="0.1 0.1 0.05" />
+      </geometry>
+    </collision>
+    <xacro:inertial_box mass="2.0" x="0.1" y="0.1" z="0.1">
+      <origin xyz="0 0 0.025" />
+    </xacro:inertial_box>
+  </link>
   <joint name="base_joint" type="continuous">
     <parent link="base_link" />

Commit message: Patch: - Added `gazebo.xacro` to `robot.urdf.xacro` for Joint State Publication.

File: pendulum_description/description/robot.urdf.xacro (robot description, xacro)
@@ -2,9 +2,10 @@
 <robot xmlns:xacro="http://www.ros.org/wiki/xacro" name="pendulum">
   <xacro:include filename="inertial_macros.xacro" />
+  <xacro:include filename="gazebo.xacro" />
   <link name="base_link">
     <visual>
       <origin xyz="0.0 0.0 0.025" />
       <geometry>
-        <box size="0.1 0.1 0.05" />
+        <box size="0.1 0.25 0.05" />
       </geometry>
       <material name="gray">
@@ -18,5 +19,5 @@
       </geometry>
     </collision>
-    <xacro:inertial_box mass="2.0" x="0.1" y="0.1" z="0.1">
+    <xacro:inertial_box mass="5.0" x="0.1" y="0.25" z="0.05">
       <origin xyz="0 0 0.025" />
     </xacro:inertial_box>

Commit message: Changed the urdf to match the model

File: pendulum_description/description/robot.urdf.xacro (robot description, xacro)
@@ -26,20 +26,20 @@
     <parent link="base_link" />
     <child link="pendulum_arm" />
-    <origin xyz="0 0 0.35" />
+    <origin xyz="0 0 0.5" />
   </joint>
   <link name="pendulum_arm">
     <visual>
-      <origin xyz="0.0 0.0 -0.1" />
+      <origin xyz="0.0 0.0 -0.15" />
       <geometry>
-        <cylinder radius="0.02" length="0.2" />
+        <box size="0.015 0.015 0.305" />
       </geometry>
-      <material name="blue">
-        <color rgba="0 0 1 1" />
+      <material name="grey">
+        <color rgba="0.3 0.3 0.3 1" />
       </material>
     </visual>
     <collision>
-      <origin xyz="0.0 0.0 -0.1" />
+      <origin xyz="0.0 0.0 -0.3" />
       <geometry>
-        <cylinder radius="0.02" length="0.2" />
+        <box size="0.015 0.015 0.305" />
       </geometry>
     </collision>
@@ -51,13 +51,13 @@
     <parent link="pendulum_arm" />
     <child link="pendulum_bob" />
-    <origin xyz="0 0 -0.2" />
+    <origin xyz="0 0 -0.325" />
   </joint>
   <link name="pendulum_bob">
     <visual>
       <geometry>
-        <sphere radius="0.05" />
+        <sphere radius="0.025" />
       </geometry>
-      <material name="red">
-        <color rgba="1 0 0 1" />
+      <material name="orange">
+        <color rgba="1 0.25 0 1" />
       </material>
     </visual>
