Commit message: Set default state for model to start at setpoint. Added Entity Control service to ROS for external control and reset (to be implemented)

File: pendulum_description/description/robot.urdf.xacro (robot description, xacro)
@@ -72,5 +72,5 @@
     <parent link="base_link" />
     <child link="pendulum_arm" />
-    <origin xyz="${base_length/2 + pendulum_arm_size/2} 0 0.0" />
+    <origin xyz="${base_length/2 + pendulum_arm_size/2} 0 0" rpy="0 ${pi} 0" />
   </joint>
   <link name="pendulum_arm">

Commit message: Major changes: - Removed `ros2_control` stuff again (will add it back later) - URDF format normalized with main branch - `gazebo.launch.py` now spawns bot (rebase caused accidental overwrite)

File: pendulum_description/description/robot.urdf.xacro (robot description, xacro)
@@ -40,6 +40,6 @@
   <joint name="base_joint" type="fixed">
     <parent link="base_link" />
-    <child link="holder_link" />
-    <origin xyz="0 0 0.05" rpy="0 0 0" />
+    <child link="base_rod" />
+    <origin xyz="0 0 0" rpy="0 0 ${pi}" />
   </joint>
   <link name="base_rod">
@@ -94,4 +94,5 @@
     <child link="shaft_link" />
     <origin xyz="0 0 ${(actuator_height + 0.015)/2}" rpy="0 ${pi/2} 0" />
+    <dynamics damping="1e-5" friction="0.035" />
   </joint>
   <link name="shaft_link">
@@ -182,5 +183,5 @@
       </geometry>
     </collision>
-    <xacro:inertial_box mass="0.785" x="0.05" y="0.05" z="0.05">
+    <xacro:inertial_box mass="${pendulum_mass + bob_mass}" x="0.05" y="0.05" z="0.05">
       <origin xyz="0 0 0" />
     </xacro:inertial_box>
