Commit message: New Branch (Aim: Motorized Inverted Pendulum): - Major changes to base structure `robot.urdf.xacro`. - Renamed and added all "continuous" joints to `gazebo.xacro` for `/joint_states` data.

File: pendulum_description/description/gazebo.xacro (robot description, xacro)
@@ -5,5 +5,6 @@
       name="gz::sim::systems::JointStatePublisher">
       <topic>joint_states</topic>
-      <joint_name>base_joint</joint_name>
+      <joint_name>shaft_joint</joint_name>
+      <joint_name>pendulum_joint</joint_name>
     </plugin>
   </gazebo>

File: pendulum_description/description/robot.urdf.xacro (robot description, xacro)
@@ -7,5 +7,5 @@
       <origin xyz="0.0 0.0 0.025" />
       <geometry>
-        <box size="0.1 0.25 0.05" />
+        <cylinder length="0.05" radius="0.25" />
       </geometry>
       <material name="gray">
@@ -16,40 +16,111 @@
       <origin xyz="0.0 0.0 0.025" />
       <geometry>
-        <box size="0.1 0.1 0.05" />
+        <cylinder length="0.05" radius="0.25" />
       </geometry>
     </collision>
-    <xacro:inertial_box mass="5.0" x="0.1" y="0.25" z="0.05">
+    <xacro:inertial_cylinder mass="5.0" radius="0.25" length="0.05">
       <origin xyz="0 0 0.025" />
+    </xacro:inertial_cylinder>
+  </link>
+  <joint name="base_joint" type="fixed">
+    <parent link="base_link" />
+    <child link="base_rod" />
+    <origin xyz="0 0 0.05" />
+  </joint>
+  <link name="base_rod">
+    <visual>
+      <origin xyz="0 0 0.25" />
+      <geometry>
+        <cylinder radius="0.01" length="0.5" />
+      </geometry>
+      <material name="gray">
+        <color rgba="0.5 0.5 0.5 1" />
+      </material>
+    </visual>
+    <collision>
+      <origin xyz="0 0 0.25" />
+      <geometry>
+        <cylinder radius="0.01" length="0.5" />
+      </geometry>
+    </collision>
+    <xacro:inertial_cylinder mass="1.0" radius="0.01" length="0.5">
+      <origin xyz="0 0 0.25" />
+    </xacro:inertial_cylinder>
+  </link>
+  <joint name="motor_joint" type="fixed">
+    <parent link="base_rod" />
+    <child link="motor_link" />
+    <origin xyz="0 0 0.5" />
+  </joint>
+  <link name="motor_link">
+    <visual>
+      <geometry>
+        <box size="0.1 0.1 0.1" />
+      </geometry>
+      <material name="dark_gray">
+        <color rgba="0.2 0.2 0.2 1" />
+      </material>
+    </visual>
+    <collision>
+      <geometry>
+        <box size="0.1 0.1 0.1" />
+      </geometry>
+    </collision>
+    <xacro:inertial_box mass="0.34" x="0.1" y="0.1" z="0.1">
+      <origin xyz="0 0 0.05" />
     </xacro:inertial_box>
   </link>
-  <joint name="base_joint" type="continuous">
-    <parent link="base_link" />
+  <joint name="shaft_joint" type="continuous">
+    <parent link="motor_link" />
+    <child link="shaft_link" />
+    <origin xyz="0 0 0.055" rpy="0.0 ${pi/2} 0.0" />
+  </joint>
+  <link name="shaft_link">
+    <visual>
+      <geometry>
+        <box size="0.01 0.01 0.5" />
+      </geometry>
+      <material name="light_gray">
+        <color rgba="0.8 0.8 0.8 1" />
+      </material>
+    </visual>
+    <collision>
+      <geometry>
+        <box size="0.01 0.01 0.5" />
+      </geometry>
+    </collision>
+    <xacro:inertial_box mass="0.135" x="0.01" y="0.01" z="0.5">
+      <origin xyz="0 0 0.25" />
+    </xacro:inertial_box>
+  </link>
+  <joint name="pendulum_joint" type="continuous">
+    <parent link="shaft_link" />
     <child link="pendulum_arm" />
-    <origin xyz="0 0 0.35" />
+    <origin xyz="0 0 -0.25" rpy="0.0 ${-pi/2} 0.0" />
   </joint>
   <link name="pendulum_arm">
     <visual>
-      <origin xyz="0.0 0.0 -0.1" />
+      <origin xyz="0.0 0.0 -0.2" />
       <geometry>
-        <cylinder radius="0.02" length="0.2" />
+        <box size="0.02 0.02 0.4" />
       </geometry>
-      <material name="blue">
-        <color rgba="0 0 1 1" />
+      <material name="gray">
+        <color rgba="0.5 0.5 0.5 1" />
       </material>
     </visual>
     <collision>
-      <origin xyz="0.0 0.0 -0.1" />
+      <origin xyz="0.0 0.0 -0.2" />
       <geometry>
-        <cylinder radius="0.02" length="0.2" />
+        <box size="0.02 0.02 0.4" />
       </geometry>
     </collision>
-    <xacro:inertial_cylinder mass="0.5" radius="0.02" length="0.2">
-      <origin xyz="0.0 0.0 -0.1" />
-    </xacro:inertial_cylinder>
+    <xacro:inertial_box mass="0.432" x="0.02" y="0.02" z="0.4">
+      <origin xyz="0.0 0.0 -0.2" />
+    </xacro:inertial_box>
   </link>
   <joint name="arm_to_bob" type="fixed">
     <parent link="pendulum_arm" />
     <child link="pendulum_bob" />
-    <origin xyz="0 0 -0.2" />
+    <origin xyz="0 0 -0.4" />
   </joint>
   <link name="pendulum_bob">
@@ -58,6 +129,6 @@
         <sphere radius="0.05" />
       </geometry>
-      <material name="red">
-        <color rgba="1 0 0 1" />
+      <material name="orange">
+        <color rgba="1 0.15 0 1" />
       </material>
     </visual>
@@ -67,7 +138,25 @@
       </geometry>
     </collision>
-    <xacro:inertial_sphere mass="1.0" radius="0.05">
+    <xacro:inertial_sphere mass="0.0573" radius="0.05">
       <origin xyz="0 0 0" />
     </xacro:inertial_sphere>
   </link>
+  <joint name="counterweight_joint" type="fixed">
+    <parent link="shaft_link" />
+    <child link="counterweight_link" />
+    <origin xyz="0.0 0.0 0.25" />
+  </joint>
+  <link name="counterweight_link">
+    <visual>
+      <geometry>
+        <box size="0.05 0.05 0.05" />
+      </geometry>
+      <material name="blue">
+        <color rgba="0 0 1 1" />
+      </material>
+      <xacro:inertial_box mass="0.785" x="0.05" y="0.05" z="0.05">
+        <origin xyz="0 0 0" />
+      </xacro:inertial_box>
+    </visual>
+  </link>
 </robot>

Commit message: Major changes: - Added `ros2_control` specific code, injected in URDF. - Added `pendulum_controller.yaml` for motor control. - Added `pendulum_pid` for first iteration of a PID controller, yet to implement recovery mechanisms. - Separated spawning and controller scripts into `spawn_entity.launch.py` for repeated resets without closing gazebo/RViz.

File: pendulum_description/description/gazebo.xacro (robot description, xacro)
@@ -2,4 +2,5 @@
 <robot xmlns:xacro="http://www.ros.org/wiki/xacro">
   <gazebo>
+    <!-- Joint state publisher (in-built) -->
     <plugin filename="gz-sim-joint-state-publisher-system"
       name="gz::sim::systems::JointStatePublisher">
@@ -8,4 +9,8 @@
       <joint_name>pendulum_joint</joint_name>
     </plugin>
+    <!-- ROS2 Control (needs yaml file) -->
+    <plugin filename="gz_ros2_control-system" name="gz_ros2_control::GazeboSimROS2ControlPlugin">
+      <parameters>$(find pendulum_description)/config/pendulum_controller.yaml</parameters>
+    </plugin>
   </gazebo>
 </robot>

File: pendulum_description/description/robot.urdf.xacro (robot description, xacro)
@@ -3,4 +3,5 @@
   <xacro:include filename="inertial_macros.xacro" />
   <xacro:include filename="gazebo.xacro" />
+  <xacro:include filename="ros2_control.xacro" />
   <link name="base_link">
     <visual>
@@ -71,8 +72,11 @@
     </xacro:inertial_box>
   </link>
+  <!-- Stepper moves this joint -->
   <joint name="shaft_joint" type="continuous">
     <parent link="motor_link" />
     <child link="shaft_link" />
     <origin xyz="0 0 0.055" rpy="0.0 ${pi/2} 0.0" />
+    <limit effort="2.0" velocity="6.0" />
+    <dynamics damping="0.1" friction="0.01" />
   </joint>
   <link name="shaft_link">
@@ -94,8 +98,10 @@
     </xacro:inertial_box>
   </link>
+  <!-- Encoder reads this joint -->
   <joint name="pendulum_joint" type="continuous">
     <parent link="shaft_link" />
     <child link="pendulum_arm" />
-    <origin xyz="0 0 -0.25" rpy="0.0 ${-pi/2} 0.0" />
+    <origin xyz="0 0 -0.25" rpy="0.0 ${-pi/2} ${pi}" />
+    <dynamics damping="0.05" friction="0.001" />
   </joint>
   <link name="pendulum_arm">
