Commit message: Modified setup slightly for upcoming motor control. Changes: - URDF updated to have a motor visualization, and made pendulum inverted (as it should be ;) - Gazebo plugin added for joint control (Yet to fix topic mapping - see below) - Added new bridge topic for ROS2 `joint_control` (the weird name for Gazebo works, but needs fixing; TODO) - Added *NEW* reset logic from ROS2 topic to Gazebo; currently resets when pendulum falls beyond `THRESHOLD` (run using `ros2 run pendulum_sim reset_world_node`) - Updated `setup.py` to recognise and register the new node.

File: pendulum_description/description/gazebo.xacro (robot description, xacro)
@@ -2,4 +2,5 @@
 <robot xmlns:xacro="http://www.ros.org/wiki/xacro">
   <gazebo>
+    <!-- Publish joint states -->
     <plugin filename="gz-sim-joint-state-publisher-system"
       name="gz::sim::systems::JointStatePublisher">
@@ -7,4 +8,11 @@
       <joint_name>base_joint</joint_name>
     </plugin>
+    <!-- Joint Control -->
+    <plugin
+      filename="gz-sim-apply-joint-force-system"
+      name="gz::sim::systems::ApplyJointForce">
+      <topic>joint_control</topic>
+      <joint_name>base_joint</joint_name>
+    </plugin>
   </gazebo>
 </robot>

File: pendulum_description/description/robot.urdf.xacro (robot description, xacro)
@@ -3,4 +3,18 @@
   <xacro:include filename="inertial_macros.xacro" />
   <xacro:include filename="gazebo.xacro" />
+  <!-- Variables -->
+  <xacro:property name="pendulum_height" value="0.5" />
+  <xacro:property name="actuator_radius" value="0.05" />
+  <xacro:property name="actuator_height" value="0.1" />
+  <xacro:property name="pendulum_length" value="0.305" />
+  <xacro:property name="pendulum_mass" value="0.75" />
+  <xacro:property name="bob_radius" value="0.025" />
+  <xacro:property name="bob_mass" value="0.01" />
+  <link name="world" />
+  <joint name="world_to_base" type="fixed">
+    <parent link="world" />
+    <child link="base_link" />
+    <origin xyz="0 0 0" rpy="0 0 ${pi}" />
+  </joint>
   <link name="base_link">
     <visual>
@@ -16,21 +30,74 @@
       <origin xyz="0.0 0.0 0.025" />
       <geometry>
-        <box size="0.1 0.1 0.05" />
+        <box size="0.1 0.25 0.05" />
       </geometry>
     </collision>
-    <xacro:inertial_box mass="5.0" x="0.1" y="0.25" z="0.05">
+    <xacro:inertial_box mass="1.0" x="0.1" y="0.25" z="0.05">
       <origin xyz="0 0 0.025" />
     </xacro:inertial_box>
   </link>
+  <joint name="base_to_holder" type="fixed">
+    <parent link="base_link" />
+    <child link="holder_link" />
+    <origin xyz="-${0.1/2 + 0.015/2} 0 0" rpy="0 0 0" />
+  </joint>
+  <link name="holder_link">
+    <visual>
+      <origin xyz="0.0 0.0 ${pendulum_height/2}" />
+      <geometry>
+        <box size="0.015 0.015 ${pendulum_height}" />
+      </geometry>
+      <material name="gray">
+        <color rgba="0.5 0.5 0.5 1" />
+      </material>
+    </visual>
+    <collision>
+      <origin xyz="0.0 0.0 ${pendulum_height/2}" />
+      <geometry>
+        <box size="0.015 0.015 ${pendulum_height}" />
+      </geometry>
+    </collision>
+    <xacro:inertial_box mass="0.5" x="0.015" y="0.015" z="${pendulum_height}">
+      <origin xyz="0 0 ${pendulum_height/2}" />
+    </xacro:inertial_box>
+  </link>
+  <joint name="holder_to_actuator" type="fixed">
+    <parent link="holder_link" />
+    <child link="actuator_link" />
+    <origin xyz="0 0 ${pendulum_height}" rpy="0 ${pi/2} 0" />
+  </joint>
+  <link name="actuator_link">
+    <visual>
+      <origin xyz="0.0 0.0 0.0" />
+      <geometry>
+        <cylinder radius="${actuator_radius}" length="${actuator_height}" />
+      </geometry>
+      <material name="blue">
+        <color rgba="0 0 1 1" />
+      </material>
+    </visual>
+    <collision>
+      <origin xyz="0.0 0.0 0.0" />
+      <geometry>
+        <cylinder radius="${actuator_radius}" length="${actuator_height}" />
+      </geometry>
+    </collision>
+    <xacro:inertial_cylinder mass="0.5" radius="${actuator_radius}" length="${actuator_height}">
+      <origin xyz="0 0 0" />
+    </xacro:inertial_cylinder>
+  </link>
+  <!-- TODO (optional assignment): Update this joint to start from `actuator_link` -->
+  <!-- And update the name to `actuator_joint` throughout the project. -->
   <joint name="base_joint" type="continuous">
     <parent link="base_link" />
     <child link="pendulum_arm" />
-    <origin xyz="0 0 0.5" />
+    <origin xyz="0 0 ${pendulum_height}" rpy="${pi} 0 0" />
+    <dynamics damping="1e-5" friction="0.035" />
   </joint>
   <link name="pendulum_arm">
     <visual>
-      <origin xyz="0.0 0.0 -0.15" />
+      <origin xyz="0.0 0.0 ${-pendulum_length / 2}" />
       <geometry>
-        <box size="0.015 0.015 0.305" />
+        <box size="0.015 0.015 ${pendulum_length}" />
       </geometry>
       <material name="grey">
@@ -39,22 +106,22 @@
     </visual>
     <collision>
-      <origin xyz="0.0 0.0 -0.3" />
+      <origin xyz="0.0 0.0 ${-pendulum_length / 2}" />
       <geometry>
-        <box size="0.015 0.015 0.305" />
+        <box size="0.015 0.015 ${pendulum_length}" />
       </geometry>
     </collision>
-    <xacro:inertial_cylinder mass="0.5" radius="0.02" length="0.2">
-      <origin xyz="0.0 0.0 -0.1" />
-    </xacro:inertial_cylinder>
+    <xacro:inertial_box mass="0.5" x="0.015" y="0.015" z="${pendulum_length}">
+      <origin xyz="0 0 ${-pendulum_length / 2}" />
+    </xacro:inertial_box>
   </link>
   <joint name="arm_to_bob" type="fixed">
     <parent link="pendulum_arm" />
     <child link="pendulum_bob" />
-    <origin xyz="0 0 -0.325" />
+    <origin xyz="0 0 ${-pendulum_length}" />
   </joint>
   <link name="pendulum_bob">
     <visual>
       <geometry>
-        <sphere radius="0.025" />
+        <sphere radius="${bob_radius}" />
       </geometry>
       <material name="orange">
@@ -64,8 +131,8 @@
     <collision>
       <geometry>
-        <sphere radius="0.05" />
+        <sphere radius="${bob_radius}" />
       </geometry>
     </collision>
-    <xacro:inertial_sphere mass="1.0" radius="0.05">
+    <xacro:inertial_sphere mass="${bob_mass}" radius="${bob_radius}">
       <origin xyz="0 0 0" />
     </xacro:inertial_sphere>

Commit message: Major changes: - Updated tests to be compatible with some jazzy/lyrical lib names. - Updated `urdf_view` in RViz to better match GazeboSim. - Updated URDF to have consistent naming. - Updated `pid_controller.py` to trigger resets once angle is exceeded, rather than separate node. - `reset_node` now integrated with `gazebo.launch.py`; topic: `/world/reset`

File: pendulum_description/description/gazebo.xacro (robot description, xacro)
@@ -6,5 +6,5 @@
       name="gz::sim::systems::JointStatePublisher">
       <topic>joint_states</topic>
-      <joint_name>base_joint</joint_name>
+      <joint_name>pendulum_joint</joint_name>
     </plugin>
     <!-- Joint Control -->
@@ -13,5 +13,5 @@
       name="gz::sim::systems::ApplyJointForce">
       <topic>joint_control</topic>
-      <joint_name>base_joint</joint_name>
+      <joint_name>pendulum_joint</joint_name>
     </plugin>
   </gazebo>

File: pendulum_description/description/robot.urdf.xacro (robot description, xacro)
@@ -15,5 +15,5 @@
     <parent link="world" />
     <child link="base_link" />
-    <origin xyz="0 0 0" rpy="0 0 ${pi}" />
+    <origin xyz="0 0 0" rpy="0 0 0" />
   </joint>
   <link name="base_link">
@@ -37,10 +37,10 @@
     </xacro:inertial_box>
   </link>
-  <joint name="base_to_holder" type="fixed">
+  <joint name="base_joint" type="fixed">
     <parent link="base_link" />
-    <child link="holder_link" />
-    <origin xyz="-${0.1/2 + 0.015/2} 0 0" rpy="0 0 0" />
+    <child link="base_rod" />
+    <origin xyz="${0.1/2 + 0.015/2} 0 0" rpy="0 0 ${pi}" />
   </joint>
-  <link name="holder_link">
+  <link name="base_rod">
     <visual>
       <origin xyz="0.0 0.0 ${pendulum_height/2}" />
@@ -58,14 +58,14 @@
       </geometry>
     </collision>
-    <xacro:inertial_box mass="0.5" x="0.015" y="0.015" z="${pendulum_height}">
+    <xacro:inertial_box mass="${pendulum_mass}" x="0.015" y="0.015" z="${pendulum_height}">
       <origin xyz="0 0 ${pendulum_height/2}" />
     </xacro:inertial_box>
   </link>
-  <joint name="holder_to_actuator" type="fixed">
-    <parent link="holder_link" />
-    <child link="actuator_link" />
+  <joint name="motor_joint" type="fixed">
+    <parent link="base_rod" />
+    <child link="motor_link" />
     <origin xyz="0 0 ${pendulum_height}" rpy="0 ${pi/2} 0" />
   </joint>
-  <link name="actuator_link">
+  <link name="motor_link">
     <visual>
       <origin xyz="0.0 0.0 0.0" />
@@ -87,10 +87,8 @@
     </xacro:inertial_cylinder>
   </link>
-  <!-- TODO (optional assignment): Update this joint to start from `actuator_link` -->
-  <!-- And update the name to `actuator_joint` throughout the project. -->
-  <joint name="base_joint" type="continuous">
-    <parent link="base_link" />
+  <joint name="pendulum_joint" type="continuous">
+    <parent link="motor_link" />
     <child link="pendulum_arm" />
-    <origin xyz="0 0 ${pendulum_height}" rpy="${pi} 0 0" />
+    <origin xyz="0 0 ${(actuator_height + 0.015)/2}" rpy="0 ${pi/2} 0" />
     <dynamics damping="1e-5" friction="0.035" />
   </joint>
@@ -111,5 +109,5 @@
       </geometry>
     </collision>
-    <xacro:inertial_box mass="0.5" x="0.015" y="0.015" z="${pendulum_length}">
+    <xacro:inertial_box mass="${pendulum_mass}" x="0.015" y="0.015" z="${pendulum_length}">
       <origin xyz="0 0 ${-pendulum_length / 2}" />
     </xacro:inertial_box>

Commit message: Minor Changes: - Modified  to publish two joints' states - Modified  to represent the intended bot

File: pendulum_description/description/gazebo.xacro (robot description, xacro)
@@ -6,4 +6,5 @@
       name="gz::sim::systems::JointStatePublisher">
       <topic>joint_states</topic>
+      <joint_name>shaft_joint</joint_name>
       <joint_name>pendulum_joint</joint_name>
     </plugin>

File: pendulum_description/description/robot.urdf.xacro (robot description, xacro)
@@ -5,6 +5,7 @@
   <!-- Variables -->
   <xacro:property name="pendulum_height" value="0.5" />
-  <xacro:property name="actuator_radius" value="0.05" />
+  <xacro:property name="actuator_radius" value="0.1" />
   <xacro:property name="actuator_height" value="0.1" />
+  <xacro:property name="shaft_length" value="0.5" />
   <xacro:property name="pendulum_length" value="0.305" />
   <xacro:property name="pendulum_mass" value="0.75" />
@@ -21,5 +22,5 @@
       <origin xyz="0.0 0.0 0.025" />
       <geometry>
-        <box size="0.1 0.25 0.05" />
+        <cylinder length="0.05" radius="0.25" />
       </geometry>
       <material name="gray">
@@ -30,15 +31,15 @@
       <origin xyz="0.0 0.0 0.025" />
       <geometry>
-        <box size="0.1 0.25 0.05" />
+        <cylinder length="0.05" radius="0.25" />
       </geometry>
     </collision>
-    <xacro:inertial_box mass="1.0" x="0.1" y="0.25" z="0.05">
+    <xacro:inertial_cylinder mass="5.0" radius="0.25" length="0.05">
       <origin xyz="0 0 0.025" />
-    </xacro:inertial_box>
+    </xacro:inertial_cylinder>
   </link>
   <joint name="base_joint" type="fixed">
     <parent link="base_link" />
-    <child link="base_rod" />
-    <origin xyz="${0.1/2 + 0.015/2} 0 0" rpy="0 0 ${pi}" />
+    <child link="holder_link" />
+    <origin xyz="0 0 0.05" rpy="0 0 0" />
   </joint>
   <link name="base_rod">
@@ -65,5 +66,5 @@
     <parent link="base_rod" />
     <child link="motor_link" />
-    <origin xyz="0 0 ${pendulum_height}" rpy="0 ${pi/2} 0" />
+    <origin xyz="0 0 ${pendulum_height}" rpy="0 0 0" />
   </joint>
   <link name="motor_link">
@@ -71,8 +72,8 @@
       <origin xyz="0.0 0.0 0.0" />
       <geometry>
-        <cylinder radius="${actuator_radius}" length="${actuator_height}" />
+        <box size="${actuator_radius} ${actuator_radius} ${actuator_height}" />
       </geometry>
-      <material name="blue">
-        <color rgba="0 0 1 1" />
+      <material name="gray">
+        <color rgba="0.5 0.5 0.5 1" />
       </material>
     </visual>
@@ -80,15 +81,41 @@
       <origin xyz="0.0 0.0 0.0" />
       <geometry>
-        <cylinder radius="${actuator_radius}" length="${actuator_height}" />
+        <box size="${actuator_radius} ${actuator_radius} ${actuator_height}" />
       </geometry>
     </collision>
-    <xacro:inertial_cylinder mass="0.5" radius="${actuator_radius}" length="${actuator_height}">
+    <xacro:inertial_box mass="0.432" x="${actuator_radius}" y="${actuator_radius}"
+      z="${actuator_height}">
+      <origin xyz="0.0 0.0 0.0" />
+    </xacro:inertial_box>
+  </link>
+  <!-- *Stepper moves this joint -->
+  <joint name="shaft_joint" type="continuous">
+    <parent link="motor_link" />
+    <child link="shaft_link" />
+    <origin xyz="0 0 ${(actuator_height + 0.015)/2}" rpy="0 ${pi/2} 0" />
+  </joint>
+  <link name="shaft_link">
+    <visual>
+      <geometry>
+        <box size="0.015 0.015 ${shaft_length}" />
+      </geometry>
+      <material name="light_gray">
+        <color rgba="0.8 0.8 0.8 1" />
+      </material>
+    </visual>
+    <collision>
+      <geometry>
+        <box size="0.015 0.015 ${shaft_length}" />
+      </geometry>
+    </collision>
+    <xacro:inertial_box mass="0.135" x="0.015" y="0.015" z="${shaft_length}">
       <origin xyz="0 0 0" />
-    </xacro:inertial_cylinder>
+    </xacro:inertial_box>
   </link>
+  <!-- *Encoder reads this joint -->
   <joint name="pendulum_joint" type="continuous">
-    <parent link="motor_link" />
+    <parent link="shaft_link" />
     <child link="pendulum_arm" />
-    <origin xyz="0 0 ${(actuator_height + 0.015)/2}" rpy="0 ${pi/2} 0" />
+    <origin xyz="0 0 ${(shaft_length + 0.015)/2}" rpy="0 ${pi/2} 0" />
     <dynamics damping="1e-5" friction="0.035" />
   </joint>
@@ -116,5 +143,5 @@
     <parent link="pendulum_arm" />
     <child link="pendulum_bob" />
-    <origin xyz="0 0 ${-pendulum_length}" />
+    <origin xyz="0 0 -${pendulum_length}" />
   </joint>
   <link name="pendulum_bob">
@@ -124,5 +151,5 @@
       </geometry>
       <material name="orange">
-        <color rgba="1 0.25 0 1" />
+        <color rgba="1 0.15 0 1" />
       </material>
     </visual>
@@ -136,3 +163,26 @@
     </xacro:inertial_sphere>
   </link>
+  <joint name="counterweight_joint" type="fixed">
+    <parent link="shaft_link" />
+    <child link="counterweight_link" />
+    <origin xyz="0.0 0.0 -${shaft_length/2}" />
+  </joint>
+  <link name="counterweight_link">
+    <visual>
+      <geometry>
+        <box size="0.05 0.05 0.05" />
+      </geometry>
+      <material name="blue">
+        <color rgba="0 0 1 1" />
+      </material>
+    </visual>
+    <collision>
+      <geometry>
+        <box size="0.05 0.05 0.05" />
+      </geometry>
+    </collision>
+    <xacro:inertial_box mass="0.785" x="0.05" y="0.05" z="0.05">
+      <origin xyz="0 0 0" />
+    </xacro:inertial_box>
+  </link>
 </robot>
