Commit message: Modified the model to a rail-based system: - Now `base_joint` is sensor only, so it is a passive joint affected by Physics. - This means `rail_joint` is an active joint, where forces will be applied. Tests Passed: - `urdf.launch.py`

File: pendulum_description/description/inertial_macros.xacro (robot description, xacro)
@@ -13,6 +13,9 @@
     </inertial>
   </xacro:macro>
-  <xacro:macro name="inertial_box" params="mass x y z *origin">
+  <xacro:macro name="inertial_box" params="mass size *origin">
     <inertial>
+      <xacro:property name="x" value="${size.split(' ')[0]}" />
+      <xacro:property name="y" value="${size.split(' ')[1]}" />
+      <xacro:property name="z" value="${size.split(' ')[2]}" />
       <xacro:insert_block name="origin" />
       <mass value="${mass}" />

File: pendulum_description/description/robot.urdf.xacro (robot description, xacro)
@@ -3,9 +3,27 @@
   <xacro:include filename="inertial_macros.xacro" />
   <xacro:include filename="gazebo.xacro" />
-  <link name="base_link">
+  <!-- Variables -->
+  <xacro:property name="rail_height" value="0.5" />
+  <xacro:property name="rail_length" value="0.5" />
+  <xacro:property name="rail_size" value="0.015" />
+  <xacro:property name="base_radius" value="0.03" />
+  <xacro:property name="base_length" value="0.05" />
+  <xacro:property name="base_mass" value="0.1" />
+  <xacro:property name="pendulum_arm_length" value="0.3" />
+  <xacro:property name="pendulum_arm_size" value="0.015" />
+  <xacro:property name="pendulum_arm_mass" value="0.5" />
+  <xacro:property name="pendulum_bob_radius" value="0.03" />
+  <xacro:property name="pendulum_bob_mass" value="1.0" />
+  <link name="world" />
+  <joint name="world_joint" type="fixed">
+    <parent link="world" />
+    <child link="rail_link" />
+    <origin xyz="0 0 ${rail_height}" rpy="0 0 ${pi/2}" />
+  </joint>
+  <link name="rail_link">
     <visual>
-      <origin xyz="0.0 0.0 0.025" />
+      <origin xyz="0 0 -${rail_size/2 + base_radius}" rpy="0 ${pi/2} 0" />
       <geometry>
-        <box size="0.1 0.25 0.05" />
+        <box size="${rail_size} ${rail_size} ${rail_length}" />
       </geometry>
       <material name="gray">
@@ -14,23 +32,51 @@
     </visual>
     <collision>
-      <origin xyz="0.0 0.0 0.025" />
+      <origin xyz="0 0 -${rail_size/2 + base_radius}" rpy="0 ${pi/2} 0" />
       <geometry>
-        <box size="0.1 0.1 0.05" />
+        <box size="${rail_size} ${rail_size} ${rail_length}" />
       </geometry>
     </collision>
-    <xacro:inertial_box mass="5.0" x="0.1" y="0.25" z="0.05">
-      <origin xyz="0 0 0.025" />
+    <xacro:inertial_box mass="${base_mass}" size="${rail_size} ${rail_size} ${rail_length}">
+      <origin xyz="0 0 -${rail_size/2 + base_radius}" rpy="0 ${pi/2} 0" />
     </xacro:inertial_box>
+  </link>
+  <joint name="rail_joint" type="prismatic">
+    <parent link="rail_link" />
+    <child link="base_link" />
+    <origin xyz="0 0 0" rpy="0 0 ${-pi/2}" />
+    <axis xyz="0 1 0" />
+    <limit effort="100" velocity="0.5" lower="${-rail_length/2}" upper="${rail_length/2}" />
+  </joint>
+  <link name="base_link">
+    <visual>
+      <origin xyz="0.0 0.0 0.0" rpy="0 ${pi/2} 0" />
+      <geometry>
+        <cylinder radius="${base_radius}" length="${base_length}" />
+      </geometry>
+      <material name="light_blue">
+        <color rgba="0.1 0.1 1 1" />
+      </material>
+    </visual>
+    <collision>
+      <origin xyz="0.0 0.0 0.0" rpy="0 ${pi/2} 0" />
+      <geometry>
+        <cylinder radius="${base_radius}" length="${base_length}" />
+      </geometry>
+    </collision>
+    <xacro:inertial_cylinder mass="${base_mass}" radius="${base_radius}"
+      length="${base_length}">
+      <origin xyz="0 0 0.0" rpy="0 ${pi/2} 0" />
+    </xacro:inertial_cylinder>
   </link>
   <joint name="base_joint" type="continuous">
     <parent link="base_link" />
     <child link="pendulum_arm" />
-    <origin xyz="0 0 0.5" />
+    <origin xyz="${base_length/2 + pendulum_arm_size/2} 0 0.0" />
   </joint>
   <link name="pendulum_arm">
     <visual>
-      <origin xyz="0.0 0.0 -0.15" />
+      <origin xyz="0.0 0.0 ${-pendulum_arm_length/2}" />
       <geometry>
-        <box size="0.015 0.015 0.305" />
+        <box size="${pendulum_arm_size} ${pendulum_arm_size} ${pendulum_arm_length}" />
       </geometry>
       <material name="grey">
@@ -39,22 +85,23 @@
     </visual>
     <collision>
-      <origin xyz="0.0 0.0 -0.3" />
+      <origin xyz="0.0 0.0 ${-pendulum_arm_length/2}" />
       <geometry>
-        <box size="0.015 0.015 0.305" />
+        <box size="${pendulum_arm_size} ${pendulum_arm_size} ${pendulum_arm_length}" />
       </geometry>
     </collision>
-    <xacro:inertial_cylinder mass="0.5" radius="0.02" length="0.2">
-      <origin xyz="0.0 0.0 -0.1" />
-    </xacro:inertial_cylinder>
+    <xacro:inertial_box mass="${pendulum_arm_mass}"
+      size="${pendulum_arm_size} ${pendulum_arm_size} ${pendulum_arm_length}">
+      <origin xyz="0.0 0.0 ${-pendulum_arm_length/2}" />
+    </xacro:inertial_box>
   </link>
   <joint name="arm_to_bob" type="fixed">
     <parent link="pendulum_arm" />
     <child link="pendulum_bob" />
-    <origin xyz="0 0 -0.325" />
+    <origin xyz="0 0 ${-pendulum_arm_length}" />
   </joint>
   <link name="pendulum_bob">
     <visual>
       <geometry>
-        <sphere radius="0.025" />
+        <sphere radius="${pendulum_bob_radius}" />
       </geometry>
       <material name="orange">
@@ -64,8 +111,8 @@
     <collision>
       <geometry>
-        <sphere radius="0.05" />
+        <sphere radius="${pendulum_bob_radius}" />
       </geometry>
     </collision>
-    <xacro:inertial_sphere mass="1.0" radius="0.05">
+    <xacro:inertial_sphere mass="${pendulum_bob_mass}" radius="${pendulum_bob_radius}">
       <origin xyz="0 0 0" />
     </xacro:inertial_sphere>
